File: hardware/MySoilSensorESP32.kicad_sch (KiCad schematic)
At the start: 37 parts, among them J1 Bat, J10 Bat, J11 6P4C, J13 6P4C, J15 6P4C, J16 6P4C, J17 PROGRAM, J18 DEBUG, J2 PROGRAM, J3 DEBUG, J5 6P4C, J6 6P4C, J7 6P4C, J8 6P4C, SW1 RESET, SW2 BOOT, SW3 RESET, SW4 BOOT, U1 ESP32-WROOM-32, U2 HT7833, U4 ESP32-WROOM-32

Commit message: additional reporting, updated README and REQUIREMENTS
Parts:
- added R7, R8, Rv, Rv1, Rv2, Rv3, Rv4, Rv5: 470k, symbol Device:R
Connections:
- net GND: now also R7.2, R8.2, Rv.2, Rv1.2, Rv2.2, Rv3.2, Rv4.2, Rv5.2
- net at J15.2: now also U4.7 (IO35), Rv4.1; no longer U4.12 (IO27)
- net at J15.4: now also U4.12 (IO27); no longer U4.7 (IO35)
- net at U4.10 (IO25): now also J11.4; no longer J11.2
- net at U4.11 (IO26): now also J13.4; no longer J13.2
- net at U4.26 (IO4): now also J16.4; no longer J16.2
- net at U4.5 (SENSOR_VN): now also J11.2, R8.1; no longer J11.4
- net at U4.6 (IO34): now also J13.2, Rv5.1; no longer J13.4
- net at U4.8 (IO32): now also J16.2, Rv3.1; no longer J16.4
- net at J8.2: now also J9.7 (Pin_7); no longer J9.8 (Pin_8)
- net at J8.4: now also J9.8 (Pin_8); no longer J9.7 (Pin_7)
- net at J7.2: now also J9.5 (Pin_5); no longer J9.6 (Pin_6)
- net at J7.4: now also J9.6 (Pin_6); no longer J9.5 (Pin_5)
- net at J5.2: now also J9.1 (Pin_1); no longer J9.2 (Pin_2)
- net at J5.4: now also J9.2 (Pin_2); no longer J9.1 (Pin_1)
- net at J4.1 (Pin_1), U1.5 (SENSOR_VN): now also R7.1
- net at J4.3 (Pin_3), U1.6 (IO34): now also Rv.1
- net at J4.5 (Pin_5), U1.7 (IO35): now also Rv1.1
- net at J4.7 (Pin_7), U1.8 (IO32): now also Rv2.1
- net at J6.2: now also J9.3 (Pin_3); no longer J9.4 (Pin_4)
- net at J6.4: now also J9.4 (Pin_4); no longer J9.3 (Pin_3)
Other:
- moved on the sheet: J11, J13, J15, J16, J5, J6, J7, J8, J9
